File: flux68k.kicad_sch (KiCad schematic)
At the start: 27 parts, among them J1 Conn_02x17_Odd_Even, J2 Conn_02x17_Odd_Even, J3 Conn_01x04, J4 Conn_01x04, J5 DB37_Female_MountingHoles, J6 Barrel_Jack, J7 Conn_01x01, J8 Conn_01x01, SW1 SW_SPDT, U1 74LS06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

Commit message: add missing flux68k pullups
Parts:
- added R10, R11, R12, R5, R6, R7, R8, R9: 10k, Resistor_SMD:R_0805_2012Metric_Pad1.20x1.40mm_HandSolder, symbol Device:R
- U2: value 74LS32 -> 74HCT32; Digikey 296-14891-1-ND -> 296-14868-1-ND
- U3, U4: value 74LS74 -> 74HCT74; Digikey 296-28880-1-ND -> 296-1211-1-ND
- U6: value 74LS157 -> 74HCT157; Digikey 296-14884-1-ND -> 296-31835-1-ND
Connections:
- net +5V: now also R10.1, R11.1, R12.1, R5.1, R6.1, R7.1, R8.1, R9.1
- net ~{OPTION0}: now also R5.2
- net ~{OPTION1}: now also R7.2
- net ~{OPTION2}: now also R6.2
- net ~{OPTION3}: now also R8.2
- net ~{X68K_DS0}: now also R12.2
- net ~{X68K_DS1}: now also R10.2
- net ~{X68K_DS2}: now also R11.2
- net ~{X68K_DS3}: now also R9.2
Other:
- moved on the sheet: J1, J2, J3, J4, J6, SW1, U2C, U2D, U5E, U5F

Commit message: add pullups and ideal diodes to flux68k
Parts:
- added R13: 10k, Resistor_SMD:R_0805_2012Metric_Pad1.20x1.40mm_HandSolder, symbol Device:R
- added U7, U8: MAX40200AUK, Package_TO_SOT_SMD:SOT-23-5, symbol Analog_Switch:MAX40200AUK
- J7, J8, JP1, JP2: Digikey (none) -> DNP
Connections:
- net ~{BOTTOM_DCD is gone; now on net ~{BOTTOM_DCD}: U1.9, U4.3 (C)
- net +5V: now also R13.1, U7.5 (OUT), U8.5 (OUT); no longer J6.1, SW1.3 (C)
- net GND: now also U7.2 (GND), U8.2 (GND)
- net ~{SWAP}: now reaches SW1.2 (B), U6.1 (S)
- net ~{SWAP}: now also J5.2, R13.2
- net VIN_DB37: now reaches J5.18
- net VIN_DB37: now also J5.19, U8.1 (VDD), U8.3 (EN)
- new net VIN_BARREL: J6.1, U7.1 (VDD), U7.3 (EN)
- no-connect marks 14 -> 12
Other:
- moved on the sheet: J6, R3, R4, U1A, U1B, U1C, U1D, U1E, U1F, U3A, U3B, U4A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
