File: xvi_auto_switcher/xvi_auto_switcher.kicad_pcb (KiCad board)
At the start: 2 copper layers, 45 x 102 mm, 49 parts, among them J1 DB37_Female_MountingHoles, J2 Conn_02x17_Odd_Even, J3 Conn_02x17_Odd_Even, J4 Conn_01x04_Male, J5 Conn_01x02_Male, U1 74LS157, U2 74LS07

Commit message: v1.1
Parts:
- moved J4 2.17 mm to (136.5, 85.0)
Routing:
- net /~{DS1_OUT}: track 56.5 -> 54.2 mm
- net +5V: track 141.4 -> 142.3 mm
- net GND: vias 30 -> 29
Other:
- outline, holes or cut-outs redrawn
