File: xvi_auto_switcher/xvi_auto_switcher.kicad_sch (KiCad schematic)
At the start: 20 parts, among them J1 DB37_Female_MountingHoles, J2 Conn_02x17_Odd_Even, J3 Conn_02x17_Odd_Even, J4 Conn_01x04_Male, J5 Conn_01x02_Male, U1 74LS157, U2 74LS07

Commit message: update auto switcher pcb connector positions and add caps
Parts:
- added C10, C11, C12, C13, C14, C15, C16, C17, C18, C19, C20, C21, C22, C23, C25, C27, C29, C3, C31, C33, C35, C4, C5, C6, C7, C8, C9: 47p, Capacitor_SMD:C_0603_1608Metric, symbol Device:C_Small
- added unit 6 of U2
- added unit 5 of U2
- C1, C2: footprint Capacitor_SMD:C_0805_2012Metric -> Capacitor_SMD:C_0603_1608Metric; Digikey 311-1140-1-ND -> 311-1088-1-ND
- J3: Digikey 3M161112-ND -> ED10528-ND
- J5: Digikey (none) -> DNP
- R1, R2, R3, R4, R5, R6, R7, R8, R9: footprint Resistor_SMD:R_0805_2012Metric -> Resistor_SMD:R_0603_1608Metric
Connections:
- net +5V: now also U2.11, U2.13
- net GND: now also C10.2, C11.2, C12.2, C13.2, C14.2, C15.2, C16.2, C17.2, C18.2, C19.2, C20.2, C21.2, C22.2, C23.2, C25.2, C27.2, C29.2, C3.2, C31.2, C33.2, C35.2, C4.2, C5.2, C6.2, C7.2, C8.2, C9.2
- net ~{DIR}: now also C19.1
- net ~{DISKIN}: now also C18.1
- net ~{DISKTYPE}: now also C3.1
- net ~{DS0}: now also C11.1
- net ~{DS1}: now also C13.1
- net ~{DS2}: now also C15.1
- net ~{DS3}: now also C7.1
- net ~{EJECTMASK}: now also C14.1
- net ~{EJECT}: now also C12.1
- net ~{ERRDISK}: now also C20.1
- net ~{FDDINT}: now also C22.1
- net ~{INDEX}: now also C9.1
- net ~{LEDBLINK}: now also C16.1
- net ~{MOR}: now also C17.1
- net ~{OPTION0}: now also C4.1
- net ~{OPTION1}: now also C6.1
- net ~{OPTION2}: now also C8.1
- net ~{OPTION3}: now also C10.1
- net ~{RDATA}: now also C31.1
- net ~{RDY}: now also C35.1
- net ~{SIDE}: now also C33.1
- net ~{STEP}: now also C21.1
- net ~{SWAP}: now also C5.1
- net ~{TRACK00}: now also C27.1
- net ~{WDATA}: now also C23.1
- net ~{WGATE}: now also C25.1
- net ~{WP}: now also C29.1
- no-connect marks 5 -> 7
Other:
- moved on the sheet: C1, C2, J2, J3, J4, J5, R1, R2, R3, R4, R5, R6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

Commit message: v1.1
Parts:
- J4: Digikey S9490-ND -> A112643-ND
- R1, R2, R3, R4, R5, R6, R7, R8, R9: Digikey 311-4.70KCRCT-ND -> 311-4.70KHRCT-ND
- U1: value 74LS157 -> 74HCT157; Digikey 296-14884-1-ND -> 296-31835-1-ND
Changed lines of the file:
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@@
       (effects (font (size 1.27 1.27)) hide)
     )
-    (property "Digikey" "311-4.70KCRCT-ND" (at 199.39 43.18 0)
+    (property "Digikey" "311-4.70KHRCT-ND" (at 199.39 43.18 0)
       (effects (font (size 1.27 1.27)) hide)
     )
@@
       (effects (font (size 1.27 1.27)) hide)
     )
-    (property "Digikey" "S9490-ND" (at 170.18 127 0)
+    (property "Digikey" "A112643-ND" (at 170.18 127 0)
       (effects (font (size 1.27 1.27)) hide)
     )
@@
       (effects (font (size 1.27 1.27)) hide)
     )
-    (property "Digikey" "311-4.70KCRCT-ND" (at 191.77 43.18 0)
+    (property "Digikey" "311-4.70KHRCT-ND" (at 191.77 43.18 0)
       (effects (font (size 1.27 1.27)) hide)
     )
@@
       (effects (font (size 1.27 1.27)) hide)
     )
-    (property "Digikey" "311-4.70KCRCT-ND" (at 214.63 43.18 0)
+    (property "Digikey" "311-4.70KHRCT-ND" (at 214.63 43.18 0)
       (effects (font (size 1.27 1.27)) hide)
     )
@@
       (effects (font (size 1.27 1.27)) hide)
     )
-    (property "Digikey" "311-4.70KCRCT-ND" (at 161.29 58.42 0)
+    (property "Digikey" "311-4.70KHRCT-ND" (at 161.29 58.42 0)
       (effects (font (size 1.27 1.27)) hide)
     )
@@
       (effects (font (size 1.27 1.27)) hide)
     )
-    (property "Digikey" "311-4.70KCRCT-ND" (at 207.01 43.18 0)
+    (property "Digikey" "311-4.70KHRCT-ND" (at 207.01 43.18 0)
       (effects (font (size 1.27 1.27)) hide)
     )
@@
       (effects (font (size 1.27 1.27)) hide)
     )
-    (property "Digikey" "311-4.70KCRCT-ND" (at 176.53 58.42 0)
+    (property "Digikey" "311-4.70KHRCT-ND" (at 176.53 58.42 0)
       (effects (font (size 1.27 1.27)) hide)
     )
@@
       (effects (font (size 1.27 1.27)) (justify left))
     )
-    (property "Value" "74LS157" (at 243.3194 45.8271 0)
+    (property "Value" "74HCT157" (at 243.3194 45.8271 0)
       (effects (font (size 1.27 1.27)) (justify left))
     )
@@
       (effects (font (size 1.27 1.27)) hide)
     )
-    (property "Digikey" "296-14884-1-ND" (at 241.3 64.77 0)
+    (property "Digikey" "296-31835-1-ND" (at 241.3 64.77 0)
       (effects (font (size 1.27 1.27)) hide)
     )
@@
       (effects (font (size 1.27 1.27)) hide)
     )
-    (property "Digikey" "311-4.70KCRCT-ND" (at 168.91 58.42 0)
+    (property "Digikey" "311-4.70KHRCT-ND" (at 168.91 58.42 0)
       (effects (font (size 1.27 1.27)) hide)
     )
@@
       (effects (font (size 1.27 1.27)) hide)
     )
-    (property "Digikey" "311-4.70KCRCT-ND" (at 184.15 58.42 0)
+    (property "Digikey" "311-4.70KHRCT-ND" (at 184.15 58.42 0)
       (effects (font (size 1.27 1.27)) hide)
     )
@@
       (effects (font (size 1.27 1.27)) hide)
     )
-    (property "Digikey" "311-4.70KCRCT-ND" (at 201.93 91.44 0)
-      (effects (font (size 1.27 1.27)) hide)
-    )
+    (property "Digikey" "311-4.70KHRCT-ND" (at 201.93 91.44 0)
+      (effects (font (size 1.27 1.27)) hide)
+    )
